Commit message: Commit

File: arm.urdf (robot description, URDF)
Before this commit: robot arm, 3 links, 2 joints
Links:
- link lower_arm: geometry collision cylinder length=1.1 radius=0.05; visual cylinder length=1.1 radius=0.05
- link upper_arm: geometry collision cylinder length=1.1 radius=0.05; visual cylinder length=1.1 radius=0.05
Joints:
- joint elbow: axis 0 1 0 -> (none); origin xyz= 0 .1 -1  rpy=0 0 0 -> xyz= -1 0 -.5  rpy=0 0 0

Commit message: Commit

File: arm.urdf (robot description, URDF)
Before this commit: robot arm, 3 links, 2 joints
Joints:
- joint elbow: axis (none) ->  1 1 1; origin xyz= -1 0 -.5  rpy=0 0 0 -> xyz=0 0 -1.1 rpy=0 0 0
- joint shoulder: axis 0 1 0 ->  1 1 1; origin xyz= 0 0 .8 rpy=0 0 0 -> xyz= 0 0 .8 rpy=0 1.57 0
